Commit message: Modification

File: description/camera.xacro (robot description, xacro)
@@ -4,5 +4,5 @@
     <parent link="chassis"/>
     <child link="camera_link"/>
-    <origin xyz="0.305 0 0.08" repy="0 0 0"/>
+    <origin xyz="0.305 0 0.08" rpy="0 0 0"/>
     </joint>
     <link name="camera_link">
@@ -17,8 +17,8 @@
     <parent link="camera_link"/>
     <child link="camera_link_optical"/>
-    <origin xyz="0 0 0" repy="${-pi/2} 0 ${-pi/2}"/>
+    <origin xyz="0 0 0" rpy="${-pi/2} 0 ${-pi/2}"/>
     </joint>
     <link name="camera_link_optical"></link>
- <gazebo reference="laser_frame">
+ <gazebo reference="camera_link">
         <material>Gazebo/Red</material>
     </gazebo>

File: description/lidar.xacro (robot description, xacro)
@@ -4,5 +4,5 @@
     <parent link="chassis"/>
     <child link="laser_frame"/>
-    <origin xyz="0.1 0 0.175" repy="0 0 0"/>
+    <origin xyz="0.1 0 0.175" rpy="0 0 0"/>
     </joint>
     <link name="laser_frame">

Commit message: M

File: description/camera.xacro (robot description, xacro)
@@ -1,50 +1,64 @@
 <?xml version="1.0"?>
-<robot xmlns:xacro="http://www.ros.org/wiki/xacro"  >
+<robot xmlns:xacro="http://www.ros.org/wiki/xacro">
+    <!-- Camera Joint and Links -->
     <joint name="camera_joint" type="fixed">
-    <parent link="chassis"/>
-    <child link="camera_link"/>
-    <origin xyz="0.305 0 0.08" rpy="0 0 0"/>
+        <parent link="chassis"/>
+        <child link="camera_link"/>
+        <origin xyz="0.305 0 0.08" rpy="0 0 0"/>
     </joint>
     <link name="camera_link">
-    <visual>
-<geometry>
-<box size="0.01 0.03 0.03"/>
-</geometry>
-<material name="red"/>
-</visual>
-</link>
+        <visual>
+            <geometry>
+                <box size="0.01 0.03 0.03"/>
+            </geometry>
+            <!-- Corrected material name to Gazebo/Red -->
+            <material name="Gazebo/Red"/>
+        </visual>
+    </link>
     <joint name="camera_optical_joint" type="fixed">
-    <parent link="camera_link"/>
-    <child link="camera_link_optical"/>
-    <origin xyz="0 0 0" rpy="${-pi/2} 0 ${-pi/2}"/>
+        <parent link="camera_link"/>
+        <child link="camera_link_optical"/>
+        <origin xyz="0 0 0" rpy="${-pi/2} 0 ${-pi/2}"/>
     </joint>
-    <link name="camera_link_optical"></link>
- <gazebo reference="camera_link">
+    <link name="camera_link_optical">
+        <!-- Optional: Add geometry or a visual for the optical link -->
+        <visual>
+            <geometry>
+                <box size="0.01 0.01 0.01"/>
+            </geometry>
+            <material name="Gazebo/Gray"/>
+        </visual>
+    </link>
+    <!-- Gazebo Material Reference for Camera Link -->
+    <gazebo reference="camera_link">
         <material>Gazebo/Red</material>
     </gazebo>
+    <!-- Uncomment the Sensor Block if needed -->
+    <!--
+    <sensor name="laser" type="ray">
+        <pose>0 0 0 0 0 0</pose>
+        <visualize>true</visualize>
+        <update_rate>10</update_rate>
+        <ray>
+            <scan>
+                <horizontal>
+                    <samples>360</samples>
+                    <min_angle>-3.14</min_angle>
+                    <max_angle>3.14</max_angle>
+                </horizontal>
+            </scan>
+            <range>
+                <min>0.3</min>
+                <max>12</max>
+            </range>
+        </ray>
+        <plugin name="laser_controller" filename="libgazebo_ros_ray_sensor.so">
+            <ros>
+                <argument>~/out:=scan</argument>
+            </ros>
+            <output_type>sensor_msgs/LaserScan</output_type>
+            <frame_name>laser_frame</frame_name>
+        </plugin>
+    </sensor>
+    -->
 </robot>
-        <!-- <sensor name="laser" type="ray"> <!--ray means a scanning lidar-->
-            <pose> 0 0 0 0 0 0 </pose>
-            <visualize>true</visualize>
-            <update_rate>10</update_rate>
-            <ray>
-                <scan>
-                    <horizontal>
-                        <samples>360</samples>
-                        <min_angle>-3.14</min_angle>
-                        <max_angle>3.14</max_angle>
-                    </horizontal>
-                </scan>
-                <range>
-                    <min>0.3</min>
-                    <max>12</max>
-                </range>
-            </ray>
-            <plugin name="laser_controller" filename="libgazebo_ros_ray_sensor.so">
-                <ros>
-                    <argument>~/out:=scan</argument>
-                </ros>
-                <output_type>sensor_msgs/LaserScan</output_type>
-                <frame_name>laser_frame</frame_name>
-            </plugin>
-        </sensor> -->

Commit message: mod

File: description/camera.xacro (robot description, xacro)
@@ -1,17 +1,15 @@
 <?xml version="1.0"?>
-<robot xmlns:xacro="http://www.ros.org/wiki/xacro">
-    <!-- Camera Joint and Links -->
+<robot xmlns:xacro="http://www.ros.org/wiki/xacro"  >
     <joint name="camera_joint" type="fixed">
-        <parent link="chassis"/>
-        <child link="camera_link"/>
-        <origin xyz="0.305 0 0.08" rpy="0 0 0"/>
+       <parent link="chassis"/>
+       <child link="camera_link"/>
+       <origin xyz="0.305 0 0.08" rpy="0 0 0"/>
     </joint>
     <link name="camera_link">
         <visual>
-            <geometry>
-                <box size="0.01 0.03 0.03"/>
-            </geometry>
-            <!-- Corrected material name to Gazebo/Red -->
-            <material name="Gazebo/Red"/>
+          <geometry>
+              <box size="0.01 0.03 0.03"/>
+          </geometry>
+          <material name="red"/>
         </visual>
     </link>
@@ -22,43 +20,32 @@
     </joint>
     <link name="camera_link_optical">
-        <!-- Optional: Add geometry or a visual for the optical link -->
-        <visual>
-            <geometry>
-                <box size="0.01 0.01 0.01"/>
-            </geometry>
-            <material name="Gazebo/Gray"/>
-        </visual>
     </link>
-    <!-- Gazebo Material Reference for Camera Link -->
-    <gazebo reference="camera_link">
+ <gazebo reference="camera_link">
         <material>Gazebo/Red</material>
     </gazebo>
-    <!-- Uncomment the Sensor Block if needed -->
-    <!--
-    <sensor name="laser" type="ray">
-        <pose>0 0 0 0 0 0</pose>
-        <visualize>true</visualize>
-        <update_rate>10</update_rate>
-        <ray>
-            <scan>
-                <horizontal>
-                    <samples>360</samples>
-                    <min_angle>-3.14</min_angle>
-                    <max_angle>3.14</max_angle>
-                </horizontal>
-            </scan>
-            <range>
-                <min>0.3</min>
-                <max>12</max>
-            </range>
-        </ray>
-        <plugin name="laser_controller" filename="libgazebo_ros_ray_sensor.so">
-            <ros>
-                <argument>~/out:=scan</argument>
-            </ros>
-            <output_type>sensor_msgs/LaserScan</output_type>
-            <frame_name>laser_frame</frame_name>
-        </plugin>
-    </sensor>
-    -->
 </robot>
+        <!-- <sensor name="laser" type="ray"> <!--ray means a scanning lidar-->
+            <pose> 0 0 0 0 0 0 </pose>
+            <visualize>true</visualize>
+            <update_rate>10</update_rate>
+            <ray>
+                <scan>
+                    <horizontal>
+                        <samples>360</samples>
+                        <min_angle>-3.14</min_angle>
+                        <max_angle>3.14</max_angle>
+                    </horizontal>
+                </scan>
+                <range>
+                    <min>0.3</min>
+                    <max>12</max>
+                </range>
+            </ray>
+            <plugin name="laser_controller" filename="libgazebo_ros_ray_sensor.so">
+                <ros>
+                    <argument>~/out:=scan</argument>
+                </ros>
+                <output_type>sensor_msgs/LaserScan</output_type>
+                <frame_name>laser_frame</frame_name>
+            </plugin>
+        </sensor> -->
