Commit message: correction

File: description/robot_core.xacro (robot description, xacro)
@@ -22,5 +22,5 @@
    <link name="chassis">
    <visual>
-   <origin xyz="0.15 0 0.075"
+   <origin xyz="0.15 0 0.075"/>
    <geometry>
    <box size="0.3 0.3 0.15"/>

Commit message: Add Wheels

File: description/robot_core.xacro (robot description, xacro)
@@ -13,6 +13,8 @@
    <color rgba="0 0 0 1" />
    </material>
+<!-- Base LINK-->
    <link name="base_link">
    </link>
+<!--Chassis LINK-->
    <joint name="chassis_joint" type="fixed">
    <parent link="base_link"/>
@@ -29,3 +31,33 @@
    </visual>
    </link>
+   <!--Left Wheel LINK-->
+<joint name="left_wheel_joint" type="continuous">
+<parent link="base_link"/>
+<child link="left_wheel"/>
+<origin xyz="0 0.175 0" rpy="-${pi/2} 0 0"/>
+<axis xyz="0 0 1"/>
+</joint>
+<link name="left_wheel"/>
+<visual>
+<geometry>
+<cylinder radius="0.05" length="0.04"/>
+</geometry>
+<material name="blue"/>
+</visual>
+</link>
+<!--Right Wheel link-->
+<joint name="right_wheel_joint" type="continuous">
+<parent link="base_link"/>
+<child link="right_wheel"/>
+<origin xyz="0 -0.175 0" rpy="${pi/2} 0 0"/>
+<axis xyz="0 0 -1"/>
+</joint>
+<link name="right_wheel"/>
+<visual>
+<geometry>
+<cylinder radius="0.05" length="0.04"/>
+</geometry>
+<material name="blue"/>
+</visual>
+</link>
 </robot>

Commit message: Correction

File: description/robot_core.xacro (robot description, xacro)
@@ -38,5 +38,5 @@
 <axis xyz="0 0 1"/>
 </joint>
-<link name="left_wheel"/>
+<link name="left_wheel">
 <visual>
 <geometry>
@@ -53,5 +53,5 @@
 <axis xyz="0 0 -1"/>
 </joint>
-<link name="right_wheel"/>
+<link name="right_wheel">
 <visual>
 <geometry>

Commit message: Ajout caster wheel

File: description/robot_core.xacro (robot description, xacro)
@@ -61,3 +61,17 @@
 </visual>
 </link>
+<!--CASTER WHEEL LINK-->
+<joint name="caster_wheel_joint" type="fixed">
+<parent link="chassis"/>
+<child link="caster_wheel"/>
+<origin xyz="0.24 0 0"/>
+</joint>
+<link name="caster_wheel">
+<visual>
+<geometry>
+<sphere radius="0.05"/>
+</geometry>
+<material name="black"/>
+</visual>
+</link>
 </robot>

Commit message: Ajout de collision

File: description/robot_core.xacro (robot description, xacro)
@@ -30,4 +30,10 @@
    <material name="white"/>
    </visual>
+   <collision>
+   <origin xyz="0.15 0 0.075"/>
+   <geometry>
+   <box size="0.3 0.3 0.15"/>
+   </geometry>
+   </collision>
    </link>
    <!--Left Wheel LINK-->
@@ -45,4 +51,9 @@
 <material name="blue"/>
 </visual>
+<collision>
+<geometry>
+<cylinder radius="0.05" length="0.04"/>
+</geometry>
+</collision>
 </link>
 <!--Right Wheel link-->
@@ -60,4 +71,9 @@
 <material name="blue"/>
 </visual>
+<collision>
+<geometry>
+<cylinder radius="0.05" length="0.04"/>
+</geometry>
+</collision>
 </link>
 <!--CASTER WHEEL LINK-->
@@ -74,4 +90,9 @@
 <material name="black"/>
 </visual>
+<collision>
+<geometry>
+<sphere radius="0.05"/>
+</geometry>
+</collision>
 </link>
 </robot>

Commit message: inertial add

File: description/robot_core.xacro (robot description, xacro)
@@ -38,4 +38,7 @@
    </geometry>
    </collision>
+   <xacro:inertial_box mass="0.5" x="0.3" y="0.3" z="0.15">
+   <origin xyz="0.15 0 0.075" rpy="0 0 0"/>
+   </xacro:inertial_box>
    </link>
    <!--Left Wheel LINK-->
@@ -58,4 +61,7 @@
 </geometry>
 </collision>
+<xacro:inertial_cylinder mass="0.1" length="0.04" radius="0.05">
+<origin xyz="0 0 0" rpy="0 0 0"/>
+</xacro:inertial_cylinder>
 </link>
 <!--Right Wheel link-->
@@ -78,4 +84,7 @@
 </geometry>
 </collision>
+<xacro:inertial_cylinder mass="0.1" length="0.04" radius="0.05">
+<origin xyz="0 0 0" rpy="0 0 0"/>
+</xacro:inertial_cylinder>
 </link>
 <!--CASTER WHEEL LINK-->
@@ -97,4 +106,7 @@
 </geometry>
 </collision>
+<xacro:inertial_sphere mass="0.1" radius="0.05">
+<origin xyz="0 0 0" rpy="0 0 0"/>
+</xacro:inertial_sphere>
 </link>
 </robot>

Commit message: Gazebo Adds

File: description/robot_core.xacro (robot description, xacro)
@@ -41,4 +41,7 @@
    </xacro:inertial_box>
    </link>
+   <gazebo reference="chassis">
+   <material>Gazebo/white</material>
+   </gazebo>
    <!--Left Wheel LINK-->
 <joint name="left_wheel_joint" type="continuous">
@@ -64,4 +67,7 @@
 </xacro:inertial_cylinder>
 </link>
+   <gazebo reference="left_wheel">
+   <material>Gazebo/blue</material>
+   </gazebo>
 <!--Right Wheel link-->
 <joint name="right_wheel_joint" type="continuous">
@@ -87,4 +93,7 @@
 </xacro:inertial_cylinder>
 </link>
+   <gazebo reference="right_wheel">
+   <material>Gazebo/blue</material>
+   </gazebo>
 <!--CASTER WHEEL LINK-->
 <joint name="caster_wheel_joint" type="fixed">
@@ -109,3 +118,6 @@
 </xacro:inertial_sphere>
 </link>
+   <gazebo reference="caster_wheel">
+   <material>Gazebo/black</material>
+   </gazebo>
 </robot>

Commit message: correction

File: description/robot_core.xacro (robot description, xacro)
@@ -42,5 +42,5 @@
    </link>
    <gazebo reference="chassis">
-   <material>Gazebo/white</material>
+   <material>Gazebo/White</material>
    </gazebo>
    <!--Left Wheel LINK-->
@@ -68,5 +68,5 @@
 </link>
    <gazebo reference="left_wheel">
-   <material>Gazebo/blue</material>
+   <material>Gazebo/Blue</material>
    </gazebo>
 <!--Right Wheel link-->
@@ -94,5 +94,5 @@
 </link>
    <gazebo reference="right_wheel">
-   <material>Gazebo/blue</material>
+   <material>Gazebo/Blue</material>
    </gazebo>
 <!--CASTER WHEEL LINK-->
@@ -119,5 +119,5 @@
 </link>
    <gazebo reference="caster_wheel">
-   <material>Gazebo/black</material>
+   <material>Gazebo/Black</material>
    </gazebo>
 </robot>

Commit message: lidar.xacro modifications

File: description/robot_core.xacro (robot description, xacro)
@@ -13,4 +13,7 @@
    <material name="black">
    <color rgba="0 0 0 1" />
+   </material>
+   <material name="red">
+   <color rgba="1 0 0 1" />
    </material>
 <!-- Base LINK-->

Commit message: Add

File: description/robot_core.xacro (robot description, xacro)
@@ -20,4 +20,10 @@
    <link name="base_link">
    </link>
+<!--Base_Footprint link-->
+<joint name="base_footprint_joint" type="fixed">
+  <parent link="base_link"/>
+  <child link="base_footprint"/>
+  <origin xyz="0 0 0" rpy="0 0 0"/>
+</joint>
 <!--Chassis LINK-->
    <joint name="chassis_joint" type="fixed">

Commit message: correction

File: description/robot_core.xacro (robot description, xacro)
@@ -26,4 +26,6 @@
   <origin xyz="0 0 0" rpy="0 0 0"/>
 </joint>
+<link name="basefootprint">
+</link>
 <!--Chassis LINK-->
    <joint name="chassis_joint" type="fixed">

Commit message: correction

File: description/robot_core.xacro (robot description, xacro)
@@ -26,5 +26,5 @@
   <origin xyz="0 0 0" rpy="0 0 0"/>
 </joint>
-<link name="basefootprint">
+<link name="base_footprint">
 </link>
 <!--Chassis LINK-->
